Commit message: added g1 simple hand ros2 control

File: unitree_robots_description/models/g1/g1_23dof.urdf (robot description, URDF)
Before this commit: robot g1_23dof, 33 links, 32 joints
Links:
- link head_link: geometry collision mesh filename=file://$(find unitree_robots_description)/models/g1/meshes/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; visual mesh filename=file://$(find unitree_robots_description)/models/g1/meshes/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
- link left_ankle_pitch_link: geometry collision mesh filename=file://$(find unitree_robots_description)/models/g1/meshes/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; visual mesh filename=file://$(find unitree_robots_description)/models/g1/meshes/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
- link left_ankle_roll_link: geometry collision sphere radius=0.005; collision sphere radius=0.005
- link left_elbow_link: geometry collision mesh filename=file://$(find unitree_robots_description)/models/g1/meshes/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; visual mesh filename=file://$(find unitree_robots_description)/models/g1/meshes/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
- link left_hip_pitch_link: geometry collision mesh filename=file://$(find unitree_robots_description)/models/g1/meshes/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; visual mesh filename=file://$(find unitree_robots_description)/models/g1/meshes/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
- link left_hip_roll_link: geometry collision mesh filename=file://$(find unitree_robots_description)/models/g1/meshes/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; visual mesh filename=file://$(find unitree_robots_description)/models/g1/meshes/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
- link left_hip_yaw_link: geometry collision mesh filename=file://$(find unitree_robots_description)/models/g1/meshes/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; visual mesh filename=file://$(find unitree_robots_description)/models/g1/meshes/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
- link left_knee_link: geometry collision mesh filename=file://$(find unitree_robots_description)/models/g1/meshes/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; visual mesh filename=file://$(find unitree_robots_description)/models/g1/meshes/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
- link left_shoulder_pitch_link: geometry collision cylinder length=0.05 radius=0.03; visual mesh filename=file://$(find unitree_robots_description)/models/g1/meshes/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
- link left_shoulder_roll_link: geometry collision cylinder length=0.03 radius=0.03; visual mesh filename=file://$(find unitree_robots_description)/models/g1/meshes/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
- link left_shoulder_yaw_link: geometry collision mesh filename=file://$(find unitree_robots_description)/models/g1/meshes/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; visual mesh filename=file://$(find unitree_robots_description)/models/g1/meshes/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
- link left_wrist_roll_rubber_hand: geometry collision mesh filename=file://$(find unitree_robots_description)/models/g1/meshes/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; visual mesh filename=file://$(find unitree_robots_description)/models/g1/meshes/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
- link logo_link: geometry collision mesh filename=file://$(find unitree_robots_description)/models/g1/meshes/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; visual mesh filename=file://$(find unitree_robots_description)/models/g1/meshes/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
- link pelvis: geometry visual mesh filename=file://$(find unitree_robots_description)/models/g1/meshes/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
- link pelvis_contour_link: geometry collision mesh filename=file://$(find unitree_robots_description)/models/g1/meshes/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; visual mesh filename=file://$(find unitree_robots_description)/models/g1/meshes/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
- link right_ankle_pitch_link: geometry collision mesh filename=file://$(find unitree_robots_description)/models/g1/meshes/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; visual mesh filename=file://$(find unitree_robots_description)/models/g1/meshes/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
- link right_ankle_roll_link: geometry collision sphere radius=0.005; collision sphere radius=0.005
- link right_elbow_link: geometry collision mesh filename=file://$(find unitree_robots_description)/models/g1/meshes/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; visual mesh filename=file://$(find unitree_robots_description)/models/g1/meshes/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
- link right_hip_pitch_link: geometry collision mesh filename=file://$(find unitree_robots_description)/models/g1/meshes/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; visual mesh filename=file://$(find unitree_robots_description)/models/g1/meshes/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
- link right_hip_roll_link: geometry collision mesh filename=file://$(find unitree_robots_description)/models/g1/meshes/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; visual mesh filename=file://$(find unitree_robots_description)/models/g1/meshes/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
- link right_hip_yaw_link: geometry collision mesh filename=file://$(find unitree_robots_description)/models/g1/meshes/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; visual mesh filename=file://$(find unitree_robots_description)/models/g1/meshes/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
- link right_knee_link: geometry collision mesh filename=file://$(find unitree_robots_description)/models/g1/meshes/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; visual mesh filename=file://$(find unitree_robots_description)/models/g1/meshes/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
- link right_shoulder_pitch_link: geometry collision cylinder length=0.05 radius=0.03; visual mesh filename=file://$(find unitree_robots_description)/models/g1/meshes/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
- link right_shoulder_roll_link: geometry collision cylinder length=0.03 radius=0.03; visual mesh filename=file://$(find unitree_robots_description)/models/g1/meshes/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
- link right_shoulder_yaw_link: geometry collision mesh filename=file://$(find unitree_robots_description)/models/g1/meshes/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; visual mesh filename=file://$(find unitree_robots_description)/models/g1/meshes/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
- link right_wrist_roll_rubber_hand: geometry collision mesh filename=file://$(find unitree_robots_description)/models/g1/meshes/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; visual mesh filename=file://$(find unitree_robots_description)/models/g1/meshes/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
- link torso_link: geometry collision mesh filename=file://$(find unitree_robots_description)/models/g1/meshes/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; visual mesh filename=file://$(find unitree_robots_description)/models/g1/meshes/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
- link waist_support_link: geometry collision mesh filename=file://$(find unitree_robots_description)/models/g1/meshes/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; visual mesh filename=file://$(find unitree_robots_description)/models/g1/meshes/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
- link waist_yaw_fixed_link: geometry visual mesh filename=file://$(find unitree_robots_description)/models/g1/meshes/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

File: unitree_robots_description/models/g1/g1_29dof_with_hand.urdf (robot description, URDF)
Before this commit: robot g1_29dof_with_hand, 54 links, 53 joints
Links:
- link head_link: geometry collision mesh filename=file://$(find unitree_robots_description)/models/g1/meshes/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; visual mesh filename=file://$(find unitree_robots_description)/models/g1/meshes/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
- link left_ankle_pitch_link: geometry collision mesh filename=file://$(find unitree_robots_description)/models/g1/meshes/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; visual mesh filename=file://$(find unitree_robots_description)/models/g1/meshes/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
- link left_ankle_roll_link: geometry collision sphere radius=0.005; collision sphere radius=0.005
- link left_elbow_link: geometry collision mesh filename=file://$(find unitree_robots_description)/models/g1/meshes/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; visual mesh filename=file://$(find unitree_robots_description)/models/g1/meshes/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
- link left_hand_index_0_link: geometry collision mesh filename=file://$(find unitree_robots_description)/models/g1/meshes/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; visual mesh filename=file://$(find unitree_robots_description)/models/g1/meshes/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
- link left_hand_index_1_link: geometry collision mesh filename=file://$(find unitree_robots_description)/models/g1/meshes/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; visual mesh filename=file://$(find unitree_robots_description)/models/g1/meshes/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
- link left_hand_middle_0_link: geometry collision mesh filename=file://$(find unitree_robots_description)/models/g1/meshes/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; visual mesh filename=file://$(find unitree_robots_description)/models/g1/meshes/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
- link left_hand_middle_1_link: geometry collision mesh filename=file://$(find unitree_robots_description)/models/g1/meshes/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; visual mesh filename=file://$(find unitree_robots_description)/models/g1/meshes/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
- link left_hand_palm_link: geometry collision mesh filename=file://$(find unitree_robots_description)/models/g1/meshes/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; visual mesh filename=file://$(find unitree_robots_description)/models/g1/meshes/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
- link left_hand_thumb_0_link: geometry collision mesh filename=file://$(find unitree_robots_description)/models/g1/meshes/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; visual mesh filename=file://$(find unitree_robots_description)/models/g1/meshes/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
- link left_hand_thumb_1_link: geometry collision box size=0.02 0.03 0.02; visual mesh filename=file://$(find unitree_robots_description)/models/g1/meshes/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
- link left_hand_thumb_2_link: geometry collision mesh filename=file://$(find unitree_robots_description)/models/g1/meshes/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; visual mesh filename=file://$(find unitree_robots_description)/models/g1/meshes/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
- link left_hip_pitch_link: geometry collision mesh filename=file://$(find unitree_robots_description)/models/g1/meshes/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; visual mesh filename=file://$(find unitree_robots_description)/models/g1/meshes/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
- link left_hip_roll_link: geometry collision mesh filename=file://$(find unitree_robots_description)/models/g1/meshes/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; visual mesh filename=file://$(find unitree_robots_description)/models/g1/meshes/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
- link left_hip_yaw_link: geometry collision mesh filename=file://$(find unitree_robots_description)/models/g1/meshes/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; visual mesh filename=file://$(find unitree_robots_description)/models/g1/meshes/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
- link left_knee_link: geometry collision mesh filename=file://$(find unitree_robots_description)/models/g1/meshes/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; visual mesh filename=file://$(find unitree_robots_description)/models/g1/meshes/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
- link left_shoulder_pitch_link: geometry collision cylinder length=0.05 radius=0.03; visual mesh filename=file://$(find unitree_robots_description)/models/g1/meshes/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
- link left_shoulder_roll_link: geometry collision cylinder length=0.03 radius=0.03; visual mesh filename=file://$(find unitree_robots_description)/models/g1/meshes/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
- link left_shoulder_yaw_link: geometry collision mesh filename=file://$(find unitree_robots_description)/models/g1/meshes/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; visual mesh filename=file://$(find unitree_robots_description)/models/g1/meshes/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
- link left_wrist_pitch_link: geometry collision mesh filename=file://$(find unitree_robots_description)/models/g1/meshes/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; visual mesh filename=file://$(find unitree_robots_description)/models/g1/meshes/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
- link left_wrist_roll_link: geometry collision mesh filename=file://$(find unitree_robots_description)/models/g1/meshes/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; visual mesh filename=file://$(find unitree_robots_description)/models/g1/meshes/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
- link left_wrist_yaw_link: geometry collision mesh filename=file://$(find unitree_robots_description)/models/g1/meshes/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; visual mesh filename=file://$(find unitree_robots_description)/models/g1/meshes/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
- link logo_link: geometry collision mesh filename=file://$(find unitree_robots_description)/models/g1/meshes/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; visual mesh filename=file://$(find unitree_robots_description)/models/g1/meshes/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
- link pelvis: geometry visual mesh filename=file://$(find unitree_robots_description)/models/g1/meshes/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
- link pelvis_contour_link: geometry collision mesh filename=file://$(find unitree_robots_description)/models/g1/meshes/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; visual mesh filename=file://$(find unitree_robots_description)/models/g1/meshes/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
- link right_ankle_pitch_link: geometry collision mesh filename=file://$(find unitree_robots_description)/models/g1/meshes/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; visual mesh filename=file://$(find unitree_robots_description)/models/g1/meshes/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
- link right_ankle_roll_link: geometry collision sphere radius=0.005; collision sphere radius=0.005
- link right_elbow_link: geometry collision mesh filename=file://$(find unitree_robots_description)/models/g1/meshes/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; visual mesh filename=file://$(find unitree_robots_description)/models/g1/meshes/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
- link right_hand_index_0_link: geometry collision mesh filename=file://$(find unitree_robots_description)/models/g1/meshes/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; visual mesh filename=file://$(find unitree_robots_description)/models/g1/meshes/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
- link right_hand_index_1_link: geometry collision mesh filename=file://$(find unitree_robots_description)/models/g1/meshes/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; visual mesh filename=file://$(find unitree_robots_description)/models/g1/meshes/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
- link right_hand_middle_0_link: geometry collision mesh filename=file://$(find unitree_robots_description)/models/g1/meshes/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; visual mesh filename=file://$(find unitree_robots_description)/models/g1/meshes/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
- link right_hand_middle_1_link: geometry collision mesh filename=file://$(find unitree_robots_description)/models/g1/meshes/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; visual mesh filename=file://$(find unitree_robots_description)/models/g1/meshes/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
- link right_hand_palm_link: geometry collision mesh filename=file://$(find unitree_robots_description)/models/g1/meshes/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; visual mesh filename=file://$(find unitree_robots_description)/models/g1/meshes/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
- link right_hand_thumb_0_link: geometry collision mesh filename=file://$(find unitree_robots_description)/models/g1/meshes/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; visual mesh filename=file://$(find unitree_robots_description)/models/g1/meshes/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
- link right_hand_thumb_1_link: geometry collision box size=0.02 0.03 0.02; visual mesh filename=file://$(find unitree_robots_description)/models/g1/meshes/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
- link right_hand_thumb_2_link: geometry collision mesh filename=file://$(find unitree_robots_description)/models/g1/meshes/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; visual mesh filename=file://$(find unitree_robots_description)/models/g1/meshes/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
- link right_hip_pitch_link: geometry collision mesh filename=file://$(find unitree_robots_description)/models/g1/meshes/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; visual mesh filename=file://$(find unitree_robots_description)/models/g1/meshes/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
- link right_hip_roll_link: geometry collision mesh filename=file://$(find unitree_robots_description)/models/g1/meshes/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; visual mesh filename=file://$(find unitree_robots_description)/models/g1/meshes/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
- link right_hip_yaw_link: geometry collision mesh filename=file://$(find unitree_robots_description)/models/g1/meshes/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; visual mesh filename=file://$(find unitree_robots_description)/models/g1/meshes/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
- link right_knee_link: geometry collision mesh filename=file://$(find unitree_robots_description)/models/g1/meshes/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; visual mesh filename=file://$(find unitree_robots_description)/models/g1/meshes/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
- link right_shoulder_pitch_link: geometry collision cylinder length=0.05 radius=0.03; visual mesh filename=file://$(find unitree_robots_description)/models/g1/meshes/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
- link right_shoulder_roll_link: geometry collision cylinder length=0.03 radius=0.03; visual mesh filename=file://$(find unitree_robots_description)/models/g1/meshes/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
- link right_shoulder_yaw_link: geometry collision mesh filename=file://$(find unitree_robots_description)/models/g1/meshes/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; visual mesh filename=file://$(find unitree_robots_description)/models/g1/meshes/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
- link right_wrist_pitch_link: geometry collision mesh filename=file://$(find unitree_robots_description)/models/g1/meshes/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; visual mesh filename=file://$(find unitree_robots_description)/models/g1/meshes/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
- link right_wrist_roll_link: geometry collision mesh filename=file://$(find unitree_robots_description)/models/g1/meshes/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; visual mesh filename=file://$(find unitree_robots_description)/models/g1/meshes/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
- link right_wrist_yaw_link: geometry collision mesh filename=file://$(find unitree_robots_description)/models/g1/meshes/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; visual mesh filename=file://$(find unitree_robots_description)/models/g1/meshes/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
- link torso_link: geometry collision mesh filename=file://$(find unitree_robots_description)/models/g1/meshes/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; visual mesh filename=file://$(find unitree_robots_description)/models/g1/meshes/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
- link waist_roll_link: geometry visual mesh filename=file://$(find unitree_robots_description)/models/g1/meshes/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
- link waist_support_link: geometry collision mesh filename=file://$(find unitree_robots_description)/models/g1/meshes/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; visual mesh filename=file://$(find unitree_robots_description)/models/g1/meshes/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
- link waist_yaw_link: geometry visual mesh filename=file://$(find unitree_robots_description)/models/g1/meshes/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
