Commit message: removed mimic joints

File: unitree_robots_description/models/g1/g1_control.xacro (robot description, xacro)
@@ -259,20 +259,4 @@
       <state_interface name="velocity"/>
     </joint>
-    <joint name="left_thumb_3_joint">
-      <command_interface name="position">
-        <param name="min">-1.57</param>
-        <param name="max">1.57</param>
-      </command_interface>
-      <state_interface name="position"/>
-      <state_interface name="velocity"/>
-    </joint>
-    <joint name="left_thumb_4_joint">
-      <command_interface name="position">
-        <param name="min">-1.57</param>
-        <param name="max">1.57</param>
-      </command_interface>
-      <state_interface name="position"/>
-      <state_interface name="velocity"/>
-    </joint>
     <joint name="left_index_1_joint">
       <command_interface name="position">
@@ -283,12 +267,4 @@
       <state_interface name="velocity"/>
     </joint>
-    <joint name="left_index_2_joint">
-      <command_interface name="position">
-        <param name="min">-1.57</param>
-        <param name="max">1.57</param>
-      </command_interface>
-      <state_interface name="position"/>
-      <state_interface name="velocity"/>
-    </joint>
     <joint name="left_middle_1_joint">
       <command_interface name="position">
@@ -299,12 +275,4 @@
       <state_interface name="velocity"/>
     </joint>
-    <joint name="left_middle_2_joint">
-      <command_interface name="position">
-        <param name="min">-1.57</param>
-        <param name="max">1.57</param>
-      </command_interface>
-      <state_interface name="position"/>
-      <state_interface name="velocity"/>
-    </joint>
     <joint name="left_ring_1_joint">
       <command_interface name="position">
@@ -315,21 +283,5 @@
       <state_interface name="velocity"/>
     </joint>
-    <joint name="left_ring_2_joint">
-      <command_interface name="position">
-        <param name="min">-1.57</param>
-        <param name="max">1.57</param>
-      </command_interface>
-      <state_interface name="position"/>
-      <state_interface name="velocity"/>
-    </joint>
     <joint name="left_little_1_joint">
-      <command_interface name="position">
-        <param name="min">-1.57</param>
-        <param name="max">1.57</param>
-      </command_interface>
-      <state_interface name="position"/>
-      <state_interface name="velocity"/>
-    </joint>
-    <joint name="left_little_2_joint">
       <command_interface name="position">
         <param name="min">-1.57</param>
@@ -356,20 +308,4 @@
       <state_interface name="velocity"/>
     </joint>
-    <joint name="right_thumb_3_joint">
-      <command_interface name="position">
-        <param name="min">-1.57</param>
-        <param name="max">1.57</param>
-      </command_interface>
-      <state_interface name="position"/>
-      <state_interface name="velocity"/>
-    </joint>
-    <joint name="right_thumb_4_joint">
-      <command_interface name="position">
-        <param name="min">-1.57</param>
-        <param name="max">1.57</param>
-      </command_interface>
-      <state_interface name="position"/>
-      <state_interface name="velocity"/>
-    </joint>
     <joint name="right_index_1_joint">
       <command_interface name="position">
@@ -380,12 +316,4 @@
       <state_interface name="velocity"/>
     </joint>
-    <joint name="right_index_2_joint">
-      <command_interface name="position">
-        <param name="min">-1.57</param>
-        <param name="max">1.57</param>
-      </command_interface>
-      <state_interface name="position"/>
-      <state_interface name="velocity"/>
-    </joint>
     <joint name="right_middle_1_joint">
       <command_interface name="position">
@@ -396,12 +324,4 @@
       <state_interface name="velocity"/>
     </joint>
-    <joint name="right_middle_2_joint">
-      <command_interface name="position">
-        <param name="min">-1.57</param>
-        <param name="max">1.57</param>
-      </command_interface>
-      <state_interface name="position"/>
-      <state_interface name="velocity"/>
-    </joint>
     <joint name="right_ring_1_joint">
       <command_interface name="position">
@@ -412,12 +332,4 @@
       <state_interface name="velocity"/>
     </joint>
-    <joint name="right_ring_2_joint">
-      <command_interface name="position">
-        <param name="min">-1.57</param>
-        <param name="max">1.57</param>
-      </command_interface>
-      <state_interface name="position"/>
-      <state_interface name="velocity"/>
-    </joint>
     <joint name="right_little_1_joint">
       <command_interface name="position">
@@ -427,13 +339,5 @@
       <state_interface name="position"/>
       <state_interface name="velocity"/>
-    </joint>
-    <joint name="right_little_2_joint">
-      <command_interface name="position">
-        <param name="min">-1.57</param>
-        <param name="max">1.57</param>
-      </command_interface>
-      <state_interface name="position"/>
-      <state_interface name="velocity"/>
-    </joint>
+    </joint>x
   </ros2_control>
   <!-- Gazebo plugins -->
