Commit message: H1 added

File: unitree_robots_description/models/h1/h1.urdf (robot description, URDF)
Before this commit: robot h1_description, 25 links, 24 joints
Links:
- link left_ankle_link: geometry collision box size=0.28 0.03 0.024; visual mesh filename=file://$(find unitree_robots_description)/models/h1/meshes/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
- link left_elbow_link: geometry collision cylinder length=0.09 radius=0.03; visual mesh filename=file://$(find unitree_robots_description)/models/h1/meshes/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
- link left_hip_pitch_link: geometry collision cylinder length=0.2 radius=0.05; visual mesh filename=file://$(find unitree_robots_description)/models/h1/meshes/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
- link left_hip_roll_link: geometry collision cylinder length=0.01 radius=0.02; visual mesh filename=file://$(find unitree_robots_description)/models/h1/meshes/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
- link left_hip_yaw_link: geometry collision cylinder length=0.02 radius=0.01; visual mesh filename=file://$(find unitree_robots_description)/models/h1/meshes/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
- link left_knee_link: geometry collision cylinder length=0.2 radius=0.05; visual mesh filename=file://$(find unitree_robots_description)/models/h1/meshes/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
- link left_shoulder_pitch_link: geometry collision cylinder length=0.04 radius=0.03; visual mesh filename=file://$(find unitree_robots_description)/models/h1/meshes/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
- link left_shoulder_roll_link: geometry collision cylinder length=0.01 radius=0.04; visual mesh filename=file://$(find unitree_robots_description)/models/h1/meshes/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
- link left_shoulder_yaw_link: geometry collision cylinder length=0.01 radius=0.04; visual mesh filename=file://$(find unitree_robots_description)/models/h1/meshes/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
- link logo_link: geometry visual mesh filename=file://$(find unitree_robots_description)/models/h1/meshes/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
- link pelvis: geometry collision sphere radius=0.05; visual mesh filename=file://$(find unitree_robots_description)/models/h1/meshes/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
- link right_ankle_link: geometry collision box size=0.28 0.03 0.024; visual mesh filename=file://$(find unitree_robots_description)/models/h1/meshes/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
- link right_elbow_link: geometry collision cylinder length=0.09 radius=0.03; visual mesh filename=file://$(find unitree_robots_description)/models/h1/meshes/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
- link right_hip_pitch_link: geometry collision cylinder length=0.2 radius=0.05; visual mesh filename=file://$(find unitree_robots_description)/models/h1/meshes/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
- link right_hip_roll_link: geometry collision cylinder length=0.01 radius=0.02; visual mesh filename=file://$(find unitree_robots_description)/models/h1/meshes/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
- link right_hip_yaw_link: geometry collision cylinder length=0.02 radius=0.01; visual mesh filename=file://$(find unitree_robots_description)/models/h1/meshes/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
- link right_knee_link: geometry collision cylinder length=0.2 radius=0.05; visual mesh filename=file://$(find unitree_robots_description)/models/h1/meshes/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
- link right_shoulder_pitch_link: geometry collision cylinder length=0.04 radius=0.03; visual mesh filename=file://$(find unitree_robots_description)/models/h1/meshes/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
- link right_shoulder_roll_link: geometry collision cylinder length=0.01 radius=0.04; visual mesh filename=file://$(find unitree_robots_description)/models/h1/meshes/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
- link right_shoulder_yaw_link: geometry collision cylinder length=0.01 radius=0.04; visual mesh filename=file://$(find unitree_robots_description)/models/h1/meshes/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
- link torso_link: geometry collision box size=0.08 0.16 0.1; visual mesh filename=file://$(find unitree_robots_description)/models/h1/meshes/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
